Commit message: fix xacro namespace prefixes

File: lwr_description/urdf/common.xacro (robot description, xacro)
@@ -23,5 +23,5 @@
  * of or in connection with the use or performance of this software.
 -->
-<robot xmlns:xacro="http://ros.org/wiki/xacro">
+<robot xmlns:xacro="http://www.ros.org/wiki/xacro">
   <!-- Directories -->
   <xacro:property name="models_path" value="package://allegro_hand_description/meshes" />
@@ -53,16 +53,16 @@
      for links.
      -->
-  <macro name="cuboid_inertia_def" params="width height length mass">
+  <xacro:macro name="cuboid_inertia_def" params="width height length mass">
     <inertia ixx="${mass * (height * height + length * length) / 12)}"
              iyy="${mass * (width * width + length * length) / 12)}"
              izz="${mass * (width * width + height * height) / 12)}"
              ixy="0" iyz="0" ixz="0"/>
-  </macro>
+  </xacro:macro>
   <!-- length is along the y-axis! -->
-  <macro name="cylinder_inertia_def" params="radius length mass">
+  <xacro:macro name="cylinder_inertia_def" params="radius length mass">
     <inertia ixx="${mass * (3 * radius * radius + length * length) / 12)}"
              iyy="${mass * radius* radius / 2)}"
              izz="${mass * (3 * radius * radius + length * length) / 12)}"
              ixy="0" iyz="0" ixz="0"/>
-  </macro>
+  </xacro:macro>
 </robot>

Commit message: fix xacro expressions

File: lwr_description/urdf/common.xacro (robot description, xacro)
@@ -54,14 +54,14 @@
      -->
   <xacro:macro name="cuboid_inertia_def" params="width height length mass">
-    <inertia ixx="${mass * (height * height + length * length) / 12)}"
-             iyy="${mass * (width * width + length * length) / 12)}"
-             izz="${mass * (width * width + height * height) / 12)}"
+    <inertia ixx="${mass * (height * height + length * length) / 12}"
+             iyy="${mass * (width * width + length * length) / 12}"
+             izz="${mass * (width * width + height * height) / 12}"
              ixy="0" iyz="0" ixz="0"/>
   </xacro:macro>
   <!-- length is along the y-axis! -->
   <xacro:macro name="cylinder_inertia_def" params="radius length mass">
-    <inertia ixx="${mass * (3 * radius * radius + length * length) / 12)}"
-             iyy="${mass * radius* radius / 2)}"
-             izz="${mass * (3 * radius * radius + length * length) / 12)}"
+    <inertia ixx="${mass * (3 * radius * radius + length * length) / 12}"
+             iyy="${mass * radius* radius / 2}"
+             izz="${mass * (3 * radius * radius + length * length) / 12}"
              ixy="0" iyz="0" ixz="0"/>
   </xacro:macro>
